File: device/interface.kicad_pcb (KiCad board)
At the start: 2 copper layers, 43.2 x 64.1 mm, 31 parts, among them IC1 ATTINY2313-S, J1 Screw_Terminal_1x02, J2 Screw_Terminal_01x02, P1 CONN_01X06, P2 CONN_02X03, P3 CONN_01X04, SW1 SW_DIP_x04, U1 L7805, U2 MAX483E, Y1 16MHz

Commit message: some changes
Parts:
- added REF**: KiCad-Logo2_8mm_SilkScreen, Symbol:KiCad-Logo2_8mm_SilkScreen, B.Cu at (119.6, 67.3)
- SW1: value SW_DIP_x04 -> ADDRESS_SW
Routing:
- net +5V: track 146.7 -> 148.4 mm
- net /RX: track 59.8 -> 60.7 mm
Other:
- board text added: "modbus-encoder v1.2"
- board text removed: "mobus-encoder v1.2"

Commit message: pcb update
Parts:
- removed REF**: KiCad-Logo2_8mm_SilkScreen, Symbol:KiCad-Logo2_8mm_SilkScreen
- added C5: 470mF, Capacitor_SMD:C_Elec_6.3x7.7, F.Cu at (127.1, 62.9)
- added C6: 0,1mF, Capacitor_SMD:C_0805_2012Metric, F.Cu at (125.2, 56.4)
- moved C3 8.21 mm to (109.5, 56.3), turned to 0 degrees
- moved U1 6.87 mm to (117.7, 60.8), turned to 90 degrees
- moved C4 0.83 mm to (109.0, 62.9)
Routing:
- net GND: track 160.3 -> 201.1 mm
- net /A1: track 43.2 -> 33.3 mm, vias 0 -> 1
- net /MISO: track 20.4 -> 25.6 mm, vias 1 -> 0
- net /MOSI: track 25.4 -> 30.3 mm, vias 1 -> 0
- net Net-(C2-Pad1): track 18.5 -> 14.7 mm
- net +24V: track 49.6 -> 46.1 mm
- net /A2: track 36.7 -> 34.5 mm
- net /RST: track 21.3 -> 23.4 mm
- net /A3: track 40.2 -> 38.3 mm
- net /PHASEA: track 35.1 -> 33.4 mm
- net +5V: track 148.4 -> 150.0 mm
- net /LED1: track 19.2 -> 17.7 mm
- net Net-(P1-Pad3): track 7.35 -> 5.95 mm, vias 1 -> 0
- net Net-(P1-Pad2): track 6.74 -> 5.94 mm, vias 1 -> 0
- net /RDE: track 46.0 -> 45.3 mm
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Other:
- board text added: "+"
- board text added: "10-30V"
- board text removed: "10-24V"

Commit message: uart pull uo
Parts:
- added R12: 10K, Resistor_SMD:R_0805_2012Metric, F.Cu at (105.5, 90.7)
- added REF**: KiCad-Logo2_8mm_SilkScreen, Symbol:KiCad-Logo2_8mm_SilkScreen, B.Cu at (117.9, 66.2)
- C4: value 47mF -> 100mF
- C5: value 470mF -> 100mF
