File: device/v1.4/interface.kicad_pcb (KiCad board)
At the start: 2 copper layers, 43.2 x 64.1 mm, 41 parts, among them IC1 ATTINY2313-S, J1 Screw_Terminal_1x02, J2 Screw_Terminal_01x02, P1 CONN_01X06, P2 CONN_02X03, P3 CONN_01X04, SW1 ADDRESS_SW, U1 L7805, U2 MAX483E, U3 PC817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

Commit message: fill zone
Routing:
- net GND: vias 0 -> 4
- added copper zone on B.Cu, net GND
Changed lines of the file:
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@@
     (thickness 1.6)
     (drawings 16)
-    (tracks 426)
+    (tracks 434)
     (zones 0)
     (modules 41)
@@
   (segment (start 111.5282 74.295) (end 111.5397 74.2835) (width 1) (layer F.Cu) (net 2))
   (segment (start 111.5397 74.2835) (end 111.5397 69.5827) (width 1) (layer F.Cu) (net 2))
-  (segment (start 117.0494 58.733) (end 117.0494 66.5596) (width 1) (layer F.Cu) (net 2))
+  (segment (start 117.0494 58.733) (end 117.0494 66.4656) (width 1) (layer F.Cu) (net 2))
   (segment (start 117.0494 66.5596) (end 114.0263 69.5827) (width 1) (layer F.Cu) (net 2))
   (segment (start 114.0263 69.5827) (end 111.5397 69.5827) (width 1) (layer F.Cu) (net 2))
@@
   (segment (start 111.5283 80.137) (end 111.5283 74.2951) (width 1) (layer F.Cu) (net 2))
   (segment (start 111.5283 74.2951) (end 111.5282 74.295) (width 1) (layer F.Cu) (net 2))
-  (segment (start 113.8287 58.733) (end 110.8487 55.753) (width 1) (layer F.Cu) (net 2))
+  (segment (start 113.8287 58.733) (end 112.44735 57.35165) (width 1) (layer F.Cu) (net 2))
   (segment (start 110.8487 55.753) (end 110.4115 55.753) (width 1) (layer F.Cu) (net 2))
-  (segment (start 124.2 58.733) (end 117.729 58.733) (width 1) (layer F.Cu) (net 2))
+  (segment (start 124.2 58.733) (end 122.242 58.733) (width 1) (layer F.Cu) (net 2))
   (segment (start 121.5937 87.0246) (end 121.5201 87.0246) (width 1) (layer F.Cu) (net 2))
   (segment (start 121.5201 87.0246) (end 120.65 86.1545) (width 1) (layer F.Cu) (net 2))
@@
   (segment (start 109.728 74.295) (end 111.5282 74.295) (width 1) (layer F.Cu) (net 2))
   (segment (start 111.506 93.5205) (end 113.538 93.5205) (width 1) (layer F.Cu) (net 2))
-  (segment (start 109.728 87.7793) (end 109.728 92.3268) (width 1) (layer F.Cu) (net 2))
+  (segment (start 109.728 87.7793) (end 109.728 88.519) (width 1) (layer F.Cu) (net 2))
   (segment (start 109.728 92.3268) (end 110.9217 93.5205) (width 1) (layer F.Cu) (net 2))
   (segment (start 110.9217 93.5205) (end 111.506 93.5205) (width 1) (layer F.Cu) (net 2))
@@
   (segment (start 123.444 95.9833) (end 124.3703 96.9096) (width 1) (layer F.Cu) (net 2))
   (segment (start 124.3703 96.9096) (end 124.3703 100.137) (width 1) (layer F.Cu) (net 2))
+  (segment (start 117.0494 66.4656) (end 117.0494 66.5596) (width 1) (layer F.Cu) (net 2))
+  (via (at 117.0494 66.4656) (size 0.8) (drill 0.4) (layers F.Cu B.Cu) (net 2))
+  (segment (start 122.242 58.733) (end 117.729 58.733) (width 1) (layer F.Cu) (net 2))
+  (via (at 122.242 58.733) (size 0.8) (drill 0.4) (layers F.Cu B.Cu) (net 2))
+  (segment (start 112.44735 57.35165) (end 110.8487 55.753) (width 1) (layer F.Cu) (net 2))
+  (via (at 112.44735 57.35165) (size 0.8) (drill 0.4) (layers F.Cu B.Cu) (net 2))
+  (segment (start 109.728 88.519) (end 109.728 92.3268) (width 1) (layer F.Cu) (net 2))
+  (via (at 109.728 88.519) (size 0.8) (drill 0.4) (layers F.Cu B.Cu) (net 2))
   (segment (start 117.348 80.137) (end 117.348 79.0117) (width 0.25) (layer F.Cu) (net 3))
   (segment (start 121.03 71.12) (end 119.7297 71.12) (width 0.25) (layer F.Cu) (net 3))
@@
   (segment (start 108.6027 71.755) (end 107.4112 72.9465) (width 0.25) (layer F.Cu) (net 32))
   (segment (start 107.4112 72.9465) (end 106.68 72.9465) (width 0.25) (layer F.Cu) (net 32))
+  (zone (net 2) (net_name GND) (layer B.Cu) (hatch edge 0.508)
+    (connect_pads (clearance 0.508))
+    (min_thickness 0.254)
+    (fill yes (arc_segments 32) (thermal_gap 0.508) (thermal_bridge_width 0.508))
+    (polygon
+      (pts
+        (xy 91.44 53.467) (xy 134.62 53.467) (xy 134.62 117.475) (xy 91.44 117.475)
+      )
+    )
+  )
 )
